File: board/nano24rf.sch (EAGLE design)
At the start: 2 parts

Commit message: with mini for lols
Parts:
- added U$3: PRO-MINI, Arduino-clone:PRO-MINI
Changed lines of the file:
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@@
 <part name="U$1" library="Arduino-clone" deviceset="NANO" device=""/>
 <part name="U$2" library="Arduino-clone" deviceset="NRF24" device=""/>
+<part name="U$3" library="Arduino-clone" deviceset="PRO-MINI" device=""/>
 </parts>
 <sheets>
@@
 <instance part="U$1" gate="G$1" x="60.96" y="50.8"/>
 <instance part="U$2" gate="G$1" x="95.25" y="60.96"/>
+<instance part="U$3" gate="G$1" x="7.62" y="58.42" rot="R180"/>
 </instances>
 <busses>

Commit message: brd
Parts:
- removed U$1: NANO, Arduino-clone:NANO
- removed U$3: PRO-MINI, Arduino-clone:PRO-MINI
- added C1: 0.1uF, ATTAMI-V0.00:CAP0805
- added C2: 1uF, ATTAMI-V0.00:CAP0805
- added D1, D2: (no value), dp_devices:DIODE-DO-214AC
- added FET1, FET2: (no value), ATTAMI-V0.00:HEADER-1X2ROUND
- added JP1, JP2: (no value), microbuilder:HEADER-1X15
- added LM317: (no value), ATTAMI-V0.00:XXX1117SOT-89
- added Q1, Q2: (no value), adafruit:MOSFET-NWAVE
- added R1, R2, R3, R4: (no value), ATTAMI-V0.00:RESISTOR0805-RES
- added SJ1: JUMPER-PAD-3-2OF3_NC_BY_TRACE_LARGE, ATTAMI-V0.00:JUMPER-PAD-3-2OF3_NC_BY_TRACE_LARGE
- added SJ2: JUMPER-PAD-2-NC_BY_TRACE, ATTAMI-V0.00:JUMPER-PAD-2-NC_BY_TRACE
- added SJ3: (no value), microbuilder:SOLDERJUMPERREFLOW
Connections:
- new net 3V3: JP1.2, U$2.VCC
- new net CE: JP2.3, U$2.CE
- new net CSN: JP2.4, U$2.CSN
- new net D3: JP2.10, R2.1
- new net D5: JP2.8, R1.1
- new net D6: JP2.7
- new net GND: C1.2, C2.2, JP1.14, JP2.12, Q1.S, Q2.S, R3.1, U$2.GND
- new net IRQ: U$2.IRQ
- new net MISO: JP2.1, U$2.MISO
- new net MOSI: JP2.2, U$2.MOSI
- new net N$1: D1.A, FET1.2, Q1.D
- new net N$2: Q1.G, R1.2
- new net N$4: D2.A, FET2.2, Q2.D
- new net N$5: Q2.G, R2.2
- new net N$7: LM317.GND, R3.2, R4.2
- new net RAW: C1.1, D1.C, D2.C, FET1.1, FET2.1, JP1.15, LM317.IN
- new net SCK: JP1.1, U$2.SCK
- new net VCC: C2.1, LM317.OUT, R4.1
Other:
- note added: "D12 D11 D10 D9 D8 D7 D6 D5 D4 D3 D2 GND RST RX TX"
- note added: "D13 3v3 AREF A0 A1 A2 A3 A4 A5 A6 A7 5V RST GND RAW"
- note added: "NANO"
- note added: "NRF24"
- note added: "http://christianto.tjahyadi.com/wp-content/uploads/2014/11/nano.jpg"

Commit message: pushed around
Parts:
- U$2: device Arduino-clone:NRF24 -> ATTAMI-V0.00:NRF24
Connections:
- net VCC renamed VOUT
Changed lines of the file:
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@@
 </classes>
 <parts>
-<part name="U$2" library="Arduino-clone" deviceset="NRF24" device=""/>
+<part name="U$2" library="ATTAMI-V0.00" deviceset="NRF24" device=""/>
 <part name="Q1" library="adafruit" deviceset="MOSFET-N" device="WAVE"/>
 <part name="D1" library="dp_devices" deviceset="DIODE" device="-DO-214AC"/>
@@
 <segment>
 <pinref part="D2" gate="D" pin="C"/>
-<wire x1="91.44" y1="2.54" x2="91.44" y2="7.62" width="0.1524" layer="91"/>
+<wire x1="91.44" y1="2.54" x2="91.44" y2="10.16" width="0.1524" layer="91"/>
 <label x="91.44" y="5.08" size="1.778" layer="95"/>
 <pinref part="FET2" gate="G$1" pin="1"/>
@@
 </segment>
 </net>
-<net name="VCC" class="0">
+<net name="VOUT" class="0">
 <segment>
 <pinref part="LM317" gate="1" pin="OUT"/>

Commit message: more jump
Connections:
- net 3V3: now also SJ1.2, SJ1.3
- net RAW: now also SJ1.1
Other:
- moved on the sheet: SJ1
Changed lines of the file:
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@@
 <text x="-2.54" y="-30.48" size="1.778" layer="91">http://christianto.tjahyadi.com/wp-content/uploads/2014/11/nano.jpg</text>
 <text x="48.26" y="71.12" size="1.778" layer="98">NANO</text>
-<text x="96.52" y="66.04" size="1.778" layer="98">NRF24</text>
+<text x="115.57" y="49.53" size="1.778" layer="98">NRF24</text>
 </plain>
 <instances>
-<instance part="U$2" gate="G$1" x="104.14" y="59.69" rot="R90"/>
+<instance part="U$2" gate="G$1" x="116.84" y="44.45" rot="R90"/>
 <instance part="Q1" gate="G$1" x="35.56" y="-10.16"/>
 <instance part="D1" gate="D" x="38.1" y="0" rot="R90"/>
@@
 <instance part="R2" gate="G$1" x="78.74" y="-12.7"/>
 <instance part="U$5" gate="1" x="27.94" y="27.94"/>
-<instance part="SJ1" gate="G$1" x="7.62" y="53.34" smashed="yes">
-<attribute name="NAME" x="10.16" y="53.721" size="1.778" layer="95"/>
+<instance part="SJ1" gate="G$1" x="106.68" y="58.42" smashed="yes" rot="R90">
+<attribute name="NAME" x="109.22" y="61.849" size="1.778" layer="95" rot="R180"/>
 </instance>
 <instance part="LM317" gate="1" x="149.86" y="5.08" smashed="yes">
@@
 <segment>
 <pinref part="U$2" gate="G$1" pin="GND"/>
-<wire x1="91.44" y1="62.23" x2="91.44" y2="68.58" width="0.1524" layer="91"/>
+<wire x1="104.14" y1="46.99" x2="104.14" y2="49.53" width="0.1524" layer="91"/>
 </segment>
 </net>
@@
 <wire x1="43.18" y1="30.48" x2="33.02" y2="30.48" width="0.1524" layer="91"/>
 <label x="33.02" y="27.94" size="1.778" layer="95"/>
+</segment>
+<segment>
+<pinref part="SJ1" gate="G$1" pin="1"/>
+<wire x1="101.6" y1="58.42" x2="99.06" y2="58.42" width="0.1524" layer="91"/>
+<label x="93.98" y="58.42" size="1.778" layer="95"/>
 </segment>
 </net>
@@
 <segment>
 <pinref part="U$2" gate="G$1" pin="VCC"/>
-<wire x1="93.98" y1="62.23" x2="93.98" y2="68.58" width="0.1524" layer="91"/>
+<wire x1="106.68" y1="46.99" x2="106.68" y2="53.34" width="0.1524" layer="91"/>
+<pinref part="SJ1" gate="G$1" pin="2"/>
+</segment>
+<segment>
+<pinref part="SJ1" gate="G$1" pin="3"/>
+<wire x1="111.76" y1="58.42" x2="114.3" y2="58.42" width="0.1524" layer="91"/>
+<label x="114.3" y="58.42" size="1.778" layer="95"/>
 </segment>
 </net>
@@
 <segment>
 <pinref part="U$2" gate="G$1" pin="MISO"/>
-<wire x1="91.44" y1="54.61" x2="90.17" y2="54.61" width="0.1524" layer="91"/>
+<wire x1="104.14" y1="39.37" x2="102.87" y2="39.37" width="0.1524" layer="91"/>
 </segment>
 <segment>
@@
 <segment>
 <pinref part="U$2" gate="G$1" pin="SCK"/>
-<wire x1="91.44" y1="57.15" x2="90.17" y2="57.15" width="0.1524" layer="91"/>
+<wire x1="104.14" y1="41.91" x2="102.87" y2="41.91" width="0.1524" layer="91"/>
 </segment>
 <segment>
@@
 <segment>
 <pinref part="U$2" gate="G$1" pin="CE"/>
-<wire x1="91.44" y1="59.69" x2="90.17" y2="59.69" width="0.1524" layer="91"/>
+<wire x1="104.14" y1="44.45" x2="102.87" y2="44.45" width="0.1524" layer="91"/>
 </segment>
 <segment>
@@
 <segment>
 <pinref part="U$2" gate="G$1" pin="CSN"/>
-<wire x1="93.98" y1="59.69" x2="95.25" y2="59.69" width="0.1524" layer="91"/>
+<wire x1="106.68" y1="44.45" x2="107.95" y2="44.45" width="0.1524" layer="91"/>
 </segment>
 <segment>
@@
 <segment>
 <pinref part="U$2" gate="G$1" pin="MOSI"/>
-<wire x1="93.98" y1="57.15" x2="95.25" y2="57.15" width="0.1524" layer="91"/>
+<wire x1="106.68" y1="41.91" x2="107.95" y2="41.91" width="0.1524" layer="91"/>
 </segment>
 <segment>
@@
 <segment>
 <pinref part="U$2" gate="G$1" pin="IRQ"/>
-<wire x1="93.98" y1="54.61" x2="95.25" y2="54.61" width="0.1524" layer="91"/>
-</segment>
-</net>
+<wire x1="106.68" y1="39.37" x2="107.95" y2="39.37" width="0.1524" layer="91"/>
+</segment>
+</net>

Commit message: add pdf, review ver
Parts:
- removed SJ2: JUMPER-PAD-2-NC_BY_TRACE, ATTAMI-V0.00:JUMPER-PAD-2-NC_BY_TRACE
- removed SJ3: (no value), microbuilder:SOLDERJUMPERREFLOW
- added SJ4: JUMPER-PAD-3-2OF3_NC_BY_TRACE_LARGE, ATTAMI-V0.00:JUMPER-PAD-3-2OF3_NC_BY_TRACE_LARGE
Connections:
- new net 5V: JP1.12, JP2.13
- new net N$6: D1.C, D2.C, FET1.1, FET2.1, SJ4.2
- net GND: now also JP1.13, JP1.3
- net RAW: now also SJ4.3; no longer D1.C, D2.C, FET1.1, FET2.1
- net VOUT: now also SJ4.1
Other:
- note added: "* 5V on the right rail should not be connected to nano! this location is originaly for a reset pin."
- note added: "D12 D11 D10 D9 D8 D7 D6 D5 D4 D3 D2 GND 5V* RX TX"
- note added: "D13 3v3 GND A0 A1 A2 A3 A4 A5 A6 A7 5V GND GND RAW"
- note added: "https://github.com/shenkarSElab/nano24rf nice nano pintout -> http://christianto.tjahyadi.com/wp-content/uploads/2014/11/nano.jpg"
- note removed: "D12 D11 D10 D9 D8 D7 D6 D5 D4 D3 D2 GND RST RX TX"
- note removed: "D13 3v3 AREF A0 A1 A2 A3 A4 A5 A6 A7 5V RST GND RAW"
- note removed: "http://christianto.tjahyadi.com/wp-content/uploads/2014/11/nano.jpg"
Changed lines of the file:
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@@
 <part name="JP1" library="microbuilder" deviceset="HEADER-1X15" device=""/>
 <part name="JP2" library="microbuilder" deviceset="HEADER-1X15" device=""/>
-<part name="SJ2" library="ATTAMI-V0.00" deviceset="JUMPER-PAD-2-NC_BY_TRACE" device=""/>
-<part name="SJ3" library="microbuilder" deviceset="SOLDERJUMPER" device="REFLOW"/>
+<part name="SJ4" library="ATTAMI-V0.00" deviceset="JUMPER-PAD-3-2OF3_NC_BY_TRACE" device="_LARGE"/>
 </parts>
 <sheets>
@@
 D2
 GND
-RST
+5V*
 RX
 TX</text>
 <text x="49.022" y="29.21" size="1.778" layer="91">D13
 3v3
-AREF
+GND
 A0
 A1
@@
 A7
 5V
-RST
+GND
 GND
 RAW</text>
-<text x="-2.54" y="-30.48" size="1.778" layer="91">http://christianto.tjahyadi.com/wp-content/uploads/2014/11/nano.jpg</text>
+<text x="-2.54" y="-38.1" size="1.778" layer="91">https://github.com/shenkarSElab/nano24rf
+nice nano pintout -&gt; http://christianto.tjahyadi.com/wp-content/uploads/2014/11/nano.jpg</text>
 <text x="48.26" y="71.12" size="1.778" layer="98">NANO</text>
 <text x="115.57" y="49.53" size="1.778" layer="98">NRF24</text>
+<text x="58.42" y="22.86" size="0.8128" layer="91">* 5V on the right rail should not be connected to nano!
+   this location is originaly for a reset pin. </text>
 </plain>
 <instances>
@@
 <instance part="JP1" gate="G$1" x="45.72" y="48.26"/>
 <instance part="JP2" gate="G$1" x="66.04" y="48.26" rot="MR0"/>
-<instance part="SJ2" gate="G$1" x="-10.16" y="53.34" smashed="yes" rot="R90">
-<attribute name="NAME" x="-12.7" y="50.8" size="1.778" layer="95" rot="R90"/>
-</instance>
-<instance part="SJ3" gate="1" x="-2.54" y="53.34" rot="R90"/>
+<instance part="SJ4" gate="G$1" x="66.04" y="15.24" smashed="yes" rot="R90">
+<attribute name="NAME" x="68.58" y="18.669" size="1.778" layer="95" rot="R180"/>
+</instance>
 </instances>
 <busses>
@@
 <pinref part="JP2" gate="G$1" pin="12"/>
 <wire x1="68.58" y1="38.1" x2="76.2" y2="38.1" width="0.1524" layer="91"/>
-<label x="73.66" y="38.1" size="1.778" layer="95"/>
 </segment>
 <segment>
 <pinref part="U$2" gate="G$1" pin="GND"/>
 <wire x1="104.14" y1="46.99" x2="104.14" y2="49.53" width="0.1524" layer="91"/>
+</segment>
+<segment>
+<pinref part="JP1" gate="G$1" pin="13"/>
+<wire x1="43.18" y1="35.56" x2="33.02" y2="35.56" width="0.1524" layer="91"/>
+</segment>
+<segment>
+<pinref part="JP1" gate="G$1" pin="3"/>
+<wire x1="43.18" y1="60.96" x2="33.02" y2="60.96" width="0.1524" layer="91"/>
 </segment>
 </net>
@@
 <net name="RAW" class="0">
 <segment>
-<pinref part="D1" gate="D" pin="C"/>
-<wire x1="38.1" y1="2.54" x2="38.1" y2="10.16" width="0.1524" layer="91"/>
-<label x="38.1" y="5.08" size="1.778" layer="95"/>
-<pinref part="FET1" gate="G$1" pin="1"/>
-<wire x1="38.1" y1="2.54" x2="50.8" y2="2.54" width="0.1524" layer="91"/>
-<junction x="38.1" y="2.54"/>
-</segment>
-<segment>
-<pinref part="D2" gate="D" pin="C"/>
-<wire x1="91.44" y1="2.54" x2="91.44" y2="10.16" width="0.1524" layer="91"/>
-<label x="91.44" y="5.08" size="1.778" layer="95"/>
-<pinref part="FET2" gate="G$1" pin="1"/>
-<wire x1="91.44" y1="2.54" x2="104.14" y2="2.54" width="0.1524" layer="91"/>
-<junction x="91.44" y="2.54"/>
-</segment>
-<segment>
 <pinref part="LM317" gate="1" pin="IN"/>
 <pinref part="C1" gate="G$1" pin="1"/>
@@
 <wire x1="101.6" y1="58.42" x2="99.06" y2="58.42" width="0.1524" layer="91"/>
 <label x="93.98" y="58.42" size="1.778" layer="95"/>
+</segment>
+<segment>
+<pinref part="SJ4" gate="G$1" pin="3"/>
+<wire x1="71.12" y1="15.24" x2="76.2" y2="15.24" width="0.1524" layer="91"/>
+<label x="73.66" y="15.24" size="1.778" layer="95"/>
 </segment>
 </net>
@@
 <label x="162.56" y="2.54" size="1.778" layer="95"/>
 </segment>
+<segment>
+<pinref part="SJ4" gate="G$1" pin="1"/>
+<wire x1="60.96" y1="15.24" x2="53.34" y2="15.24" width="0.1524" layer="91"/>
+<label x="53.34" y="15.24" size="1.778" layer="95"/>
+</segment>
 </net>
 <net name="N$7" class="0">
@@
 </segment>
 </net>
+<net name="5V" class="0">
+<segment>
+<pinref part="JP2" gate="G$1" pin="13"/>
+<wire x1="68.58" y1="35.56" x2="76.2" y2="35.56" width="0.1524" layer="91"/>
+<label x="73.66" y="35.56" size="1.778" layer="95"/>
+</segment>
+<segment>
+<pinref part="JP1" gate="G$1" pin="12"/>
+<wire x1="43.18" y1="38.1" x2="33.02" y2="38.1" width="0.1524" layer="91"/>
+</segment>
+</net>
+<net name="N$6" class="0">
+<segment>
+<pinref part="FET1" gate="G$1" pin="1"/>
+<pinref part="D1" gate="D" pin="C"/>
+<wire x1="50.8" y1="2.54" x2="38.1" y2="2.54" width="0.1524" layer="91"/>
+<wire x1="38.1" y1="2.54" x2="38.1" y2="10.16" width="0.1524" layer="91"/>
+<junction x="38.1" y="2.54"/>
+<pinref part="SJ4" gate="G$1" pin="2"/>
+<wire x1="38.1" y1="10.16" x2="66.04" y2="10.16" width="0.1524" layer="91"/>
+<pinref part="D2" gate="D" pin="C"/>
+<wire x1="66.04" y1="10.16" x2="91.44" y2="10.16" width="0.1524" layer="91"/>
+<wire x1="91.44" y1="10.16" x2="91.44" y2="2.54" width="0.1524" layer="91"/>
+<junction x="66.04" y="10.16"/>
+<pinref part="FET2" gate="G$1" pin="1"/>
+<wire x1="91.44" y1="2.54" x2="104.14" y2="2.54" width="0.1524" layer="91"/>
+<junction x="91.44" y="2.54"/>
+</segment>
+</net>

Commit message: rotate labels
Changed lines of the file:
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@@
+</nets>
+</sheet>
+<sheet>
+<plain>
+</plain>
+<instances>
+</instances>
+<busses>
+</busses>
+<nets>
 </nets>
 </sheet>

Commit message: ready for raw jumoper"
Parts:
- removed SJ4: JUMPER-PAD-3-2OF3_NC_BY_TRACE_LARGE, ATTAMI-V0.00:JUMPER-PAD-3-2OF3_NC_BY_TRACE_LARGE
- added SJ2: (no value), microbuilder:SOLDERJUMPERREFLOW
Connections:
- removed net N$6: D1.C, D2.C, FET1.1, FET2.1, SJ4.2
- net RAW: now also SJ2.1; no longer SJ4.3
- net VOUT: now also D1.C, D2.C, FET1.1, FET2.1, SJ2.2; no longer SJ4.1
Other:
- note added: "bridge this to connect RAW to mosfets"
Changed lines of the file:
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@@
 <part name="JP1" library="microbuilder" deviceset="HEADER-1X15" device=""/>
 <part name="JP2" library="microbuilder" deviceset="HEADER-1X15" device=""/>
-<part name="SJ4" library="ATTAMI-V0.00" deviceset="JUMPER-PAD-3-2OF3_NC_BY_TRACE" device="_LARGE"/>
+<part name="SJ2" library="microbuilder" deviceset="SOLDERJUMPER" device="REFLOW"/>
 </parts>
 <sheets>
@@
 <text x="58.42" y="22.86" size="0.8128" layer="91">* 5V on the right rail should not be connected to nano!
    this location is originaly for a reset pin. </text>
+<text x="132.08" y="20.32" size="1.778" layer="91">bridge this to connect RAW to mosfets</text>
 </plain>
 <instances>
@@
 <instance part="JP1" gate="G$1" x="45.72" y="48.26"/>
 <instance part="JP2" gate="G$1" x="66.04" y="48.26" rot="MR0"/>
-<instance part="SJ4" gate="G$1" x="66.04" y="15.24" smashed="yes" rot="R90">
-<attribute name="NAME" x="68.58" y="18.669" size="1.778" layer="95" rot="R180"/>
-</instance>
+<instance part="SJ2" gate="1" x="149.86" y="12.7"/>
 </instances>
 <busses>
@@
 <junction x="139.7" y="5.08"/>
 <label x="132.08" y="2.54" size="1.778" layer="95"/>
+<wire x1="139.7" y1="5.08" x2="139.7" y2="12.7" width="0.1524" layer="91"/>
+<wire x1="139.7" y1="12.7" x2="144.78" y2="12.7" width="0.1524" layer="91"/>
+<pinref part="SJ2" gate="1" pin="1"/>
 </segment>
 <segment>
@@
 <wire x1="101.6" y1="58.42" x2="99.06" y2="58.42" width="0.1524" layer="91"/>
 <label x="93.98" y="58.42" size="1.778" layer="95"/>
-</segment>
-<segment>
-<pinref part="SJ4" gate="G$1" pin="3"/>
-<wire x1="71.12" y1="15.24" x2="76.2" y2="15.24" width="0.1524" layer="91"/>
-<label x="73.66" y="15.24" size="1.778" layer="95"/>
 </segment>
 </net>
@@
 <wire x1="160.02" y1="-7.62" x2="160.02" y2="-5.08" width="0.1524" layer="91"/>
 <label x="162.56" y="2.54" size="1.778" layer="95"/>
-</segment>
-<segment>
-<pinref part="SJ4" gate="G$1" pin="1"/>
-<wire x1="60.96" y1="15.24" x2="53.34" y2="15.24" width="0.1524" layer="91"/>
-<label x="53.34" y="15.24" size="1.778" layer="95"/>
+<wire x1="160.02" y1="5.08" x2="160.02" y2="12.7" width="0.1524" layer="91"/>
+<wire x1="160.02" y1="12.7" x2="154.94" y2="12.7" width="0.1524" layer="91"/>
+<pinref part="SJ2" gate="1" pin="2"/>
+</segment>
+<segment>
+<pinref part="D2" gate="D" pin="C"/>
+<wire x1="91.44" y1="10.16" x2="91.44" y2="2.54" width="0.1524" layer="91"/>
+<pinref part="FET2" gate="G$1" pin="1"/>
+<wire x1="91.44" y1="2.54" x2="104.14" y2="2.54" width="0.1524" layer="91"/>
+<junction x="91.44" y="2.54"/>
+<label x="91.44" y="10.16" size="1.778" layer="95"/>
+</segment>
+<segment>
+<pinref part="D1" gate="D" pin="C"/>
+<pinref part="FET1" gate="G$1" pin="1"/>
+<wire x1="50.8" y1="2.54" x2="38.1" y2="2.54" width="0.1524" layer="91"/>
+<wire x1="38.1" y1="2.54" x2="38.1" y2="10.16" width="0.1524" layer="91"/>
+<junction x="38.1" y="2.54"/>
+<label x="38.1" y="10.16" size="1.778" layer="95"/>
 </segment>
 </net>
@@
 </segment>
 </net>
-<net name="N$6" class="0">
-<segment>
-<pinref part="FET1" gate="G$1" pin="1"/>
-<pinref part="D1" gate="D" pin="C"/>
-<wire x1="50.8" y1="2.54" x2="38.1" y2="2.54" width="0.1524" layer="91"/>
-<wire x1="38.1" y1="2.54" x2="38.1" y2="10.16" width="0.1524" layer="91"/>
-<junction x="38.1" y="2.54"/>
-<pinref part="SJ4" gate="G$1" pin="2"/>
-<wire x1="38.1" y1="10.16" x2="66.04" y2="10.16" width="0.1524" layer="91"/>
-<pinref part="D2" gate="D" pin="C"/>
-<wire x1="66.04" y1="10.16" x2="91.44" y2="10.16" width="0.1524" layer="91"/>
-<wire x1="91.44" y1="10.16" x2="91.44" y2="2.54" width="0.1524" layer="91"/>
-<junction x="66.04" y="10.16"/>
-<pinref part="FET2" gate="G$1" pin="1"/>
-<wire x1="91.44" y1="2.54" x2="104.14" y2="2.54" width="0.1524" layer="91"/>
-<junction x="91.44" y="2.54"/>
-</segment>
-</net>
