File: board/nanoRF.brd (EAGLE design)
At the start: 20.3 x 49.5 mm, 19 parts

Commit message: noEdge design, with gerber files
Other:
- board size 20.3 x 49.5 mm -> 22.9 x 49.5 mm
Changed lines of the file:
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@@
 <layer number="17" name="Pads" color="2" fill="1" visible="yes" active="yes"/>
 <layer number="18" name="Vias" color="2" fill="1" visible="yes" active="yes"/>
-<layer number="19" name="Unrouted" color="6" fill="1" visible="yes" active="yes"/>
+<layer number="19" name="Unrouted" color="6" fill="1" visible="no" active="yes"/>
 <layer number="20" name="Dimension" color="15" fill="1" visible="yes" active="yes"/>
 <layer number="21" name="tPlace" color="7" fill="1" visible="yes" active="yes"/>
 <layer number="22" name="bPlace" color="7" fill="1" visible="no" active="yes"/>
-<layer number="23" name="tOrigins" color="15" fill="1" visible="yes" active="yes"/>
+<layer number="23" name="tOrigins" color="15" fill="1" visible="no" active="yes"/>
 <layer number="24" name="bOrigins" color="15" fill="1" visible="no" active="yes"/>
-<layer number="25" name="tNames" color="7" fill="1" visible="yes" active="yes"/>
-<layer number="26" name="bNames" color="7" fill="1" visible="yes" active="yes"/>
-<layer number="27" name="tValues" color="7" fill="1" visible="yes" active="yes"/>
-<layer number="28" name="bValues" color="7" fill="1" visible="yes" active="yes"/>
+<layer number="25" name="tNames" color="7" fill="1" visible="no" active="yes"/>
+<layer number="26" name="bNames" color="7" fill="1" visible="no" active="yes"/>
+<layer number="27" name="tValues" color="7" fill="1" visible="no" active="yes"/>
+<layer number="28" name="bValues" color="7" fill="1" visible="no" active="yes"/>
 <layer number="29" name="tStop" color="7" fill="3" visible="no" active="yes"/>
 <layer number="30" name="bStop" color="7" fill="6" visible="no" active="yes"/>
@@
 <layer number="44" name="Drills" color="7" fill="1" visible="no" active="yes"/>
 <layer number="45" name="Holes" color="7" fill="1" visible="no" active="yes"/>
-<layer number="46" name="Milling" color="3" fill="1" visible="yes" active="yes"/>
+<layer number="46" name="Milling" color="3" fill="1" visible="no" active="yes"/>
 <layer number="47" name="Measures" color="7" fill="1" visible="no" active="yes"/>
 <layer number="48" name="Document" color="7" fill="1" visible="no" active="yes"/>
 <layer number="49" name="Reference" color="7" fill="1" visible="no" active="yes"/>
 <layer number="50" name="dxf" color="7" fill="1" visible="no" active="no"/>
-<layer number="51" name="tDocu" color="7" fill="1" visible="yes" active="yes"/>
+<layer number="51" name="tDocu" color="7" fill="1" visible="no" active="yes"/>
 <layer number="52" name="bDocu" color="7" fill="1" visible="no" active="yes"/>
 <layer number="53" name="tGND_GNDA" color="7" fill="9" visible="no" active="no"/>
@@
 <board>
 <plain>
-<wire x1="-1.27" y1="0" x2="19.05" y2="0" width="0" layer="20"/>
-<wire x1="19.05" y1="0" x2="19.05" y2="49.53" width="0" layer="20"/>
-<wire x1="19.05" y1="49.53" x2="-1.27" y2="49.53" width="0" layer="20"/>
-<wire x1="-1.27" y1="49.53" x2="-1.27" y2="0" width="0" layer="20"/>
+<wire x1="-2.54" y1="0" x2="20.32" y2="0" width="0" layer="20"/>
+<wire x1="20.32" y1="0" x2="20.32" y2="49.53" width="0" layer="20"/>
+<wire x1="20.32" y1="49.53" x2="-2.54" y2="49.53" width="0" layer="20"/>
+<wire x1="-2.54" y1="49.53" x2="-2.54" y2="0" width="0" layer="20"/>
 <text x="14.0208" y="11.7884" size="0.8128" layer="21" rot="SR45" align="top-left">TX</text>
 <text x="13.97" y="13.9982" size="0.8128" layer="21" rot="SR45" align="top-left">RX</text>
@@
 <text x="2.667" y="4.3942" size="1.016" layer="21" rot="SR270">V</text>
 <text x="13.335" y="46.99" size="1.778" layer="28" rot="MR0">idiot.io</text>
-<dimension x1="-1.27" y1="49.53" x2="19.05" y2="49.53" x3="8.89" y3="51.435" textsize="1.778" layer="51"/>
-<dimension x1="19.685" y1="49.53" x2="19.685" y2="0" x3="24.13" y3="24.765" textsize="1.778" layer="51"/>
+<dimension x1="-2.54" y1="49.53" x2="20.32" y2="49.53" x3="8.89" y3="50.8" textsize="1.778" layer="51"/>
+<dimension x1="20.32" y1="49.53" x2="20.32" y2="0" x3="26.035" y3="24.765" textsize="1.778" layer="51"/>
 </plain>
 <attributes>
@@
 <contactref element="RF24" pad="6"/>
 <polygon width="0.2032" layer="1">
-<vertex x="-1.27" y="49.403"/>
-<vertex x="-1.27" y="0"/>
-<vertex x="19.177" y="0"/>
-<vertex x="19.1516" y="49.3776"/>
+<vertex x="-2.54" y="49.53"/>
+<vertex x="-2.54" y="0"/>
+<vertex x="20.955" y="0"/>
+<vertex x="20.32" y="49.53"/>
 </polygon>
 <wire x1="16.51" y1="20.32" x2="9.525" y2="20.32" width="0.2032" layer="1"/>
@@
 <wire x1="9.017" y1="33.528" x2="8.89" y2="33.401" width="0.2032" layer="1"/>
 <polygon width="0.2032" layer="16">
-<vertex x="-1.27" y="50.292"/>
-<vertex x="-1.27" y="0"/>
-<vertex x="19.177" y="0"/>
-<vertex x="19.2278" y="50.3682"/>
+<vertex x="-2.54" y="49.657"/>
+<vertex x="-2.54" y="0"/>
+<vertex x="21.082" y="0"/>
+<vertex x="20.4978" y="49.7332"/>
 </polygon>
 <wire x1="8.89" y1="33.401" x2="8.89" y2="33.02" width="0.3048" layer="1"/>

Commit message: no edge v1.5
Parts:
- moved R5 0.13 mm to (11.4, 46.1)
- moved R6 0.13 mm to (6.35, 46.1)
Other:
- board text added: "NanoRF"
- board text added: "v1.5"
- board text removed: "nano24RF"
Changed lines of the file:
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@@
 <?xml version="1.0" encoding="utf-8"?>
 <!DOCTYPE eagle SYSTEM "eagle.dtd">
-<eagle version="8.7.0">
+<eagle version="9.0.1">
 <drawing>
 <settings>
@@
 <setting verticaltext="up"/>
 </settings>
-<grid distance="25" unitdist="mil" unit="mil" style="lines" multiple="1" display="no" altdistance="1" altunitdist="mil" altunit="mil"/>
+<grid distance="25" unitdist="mil" unit="mil" style="lines" multiple="1" display="yes" altdistance="1" altunitdist="mil" altunit="mil"/>
 <layers>
 <layer number="1" name="Top" color="4" fill="1" visible="yes" active="yes"/>
@@
 <layer number="21" name="tPlace" color="7" fill="1" visible="yes" active="yes"/>
 <layer number="22" name="bPlace" color="7" fill="1" visible="no" active="yes"/>
-<layer number="23" name="tOrigins" color="15" fill="1" visible="no" active="yes"/>
+<layer number="23" name="tOrigins" color="15" fill="1" visible="yes" active="yes"/>
 <layer number="24" name="bOrigins" color="15" fill="1" visible="no" active="yes"/>
 <layer number="25" name="tNames" color="7" fill="1" visible="no" active="yes"/>
@@
 <text x="3.3274" y="47.0944" size="0.8128" layer="21" rot="SR90">D13</text>
 <text x="3.1496" y="13.668" size="0.8128" layer="21" rot="SR90">GND</text>
-<text x="4.572" y="48.006" size="1.27" layer="21">nano24RF</text>
+<text x="4.572" y="48.006" size="1.27" layer="21">NanoRF</text>
 <rectangle x1="11.1744" y1="11.8534" x2="11.2404" y2="11.8594" layer="28" rot="R180"/>
 <rectangle x1="11.1504" y1="11.8594" x2="11.2524" y2="11.8654" layer="28" rot="R180"/>
@@
 <dimension x1="-2.54" y1="49.53" x2="20.32" y2="49.53" x3="8.89" y3="50.8" textsize="1.778" layer="51"/>
 <dimension x1="20.32" y1="49.53" x2="20.32" y2="0" x3="26.035" y3="24.765" textsize="1.778" layer="51"/>
+<text x="13.2842" y="48.133" size="1.016" layer="21" rot="R180">v1.5</text>
 </plain>
 <attributes>
@@
 <attribute name="VALUE" x="5.334" y="29.083" size="0.4064" layer="27"/>
 </element>
-<element name="R5" library="ATTAMI-V0.00" package="0805" value="" x="11.43" y="46.228" smashed="yes">
-<attribute name="VALUE" x="10.414" y="44.831" size="0.4064" layer="27"/>
+<element name="R5" library="ATTAMI-V0.00" package="0805" value="" x="11.43" y="46.101" smashed="yes">
+<attribute name="VALUE" x="10.414" y="44.704" size="0.4064" layer="27"/>
 </element>
-<element name="R6" library="ATTAMI-V0.00" package="0805" value="" x="6.35" y="46.228" smashed="yes">
-<attribute name="VALUE" x="5.334" y="44.831" size="0.4064" layer="27"/>
+<element name="R6" library="ATTAMI-V0.00" package="0805" value="" x="6.35" y="46.101" smashed="yes">
+<attribute name="VALUE" x="5.334" y="44.704" size="0.4064" layer="27"/>
 </element>
 <element name="MOSFET-34" library="nano24rf" package="FATFAD4-LONG" value="FATPAD4LONG" x="18.1102" y="5.1816" smashed="yes" rot="R90"/>
@@
 <contactref element="R6" pad="2"/>
 <wire x1="7.45" y1="43.718" x2="7.45" y2="46.028" width="0.2032" layer="1"/>
-<wire x1="7.45" y1="46.028" x2="7.25" y2="46.228" width="0.2032" layer="1" curve="90"/>
+<wire x1="7.45" y1="46.028" x2="7.25" y2="46.101" width="0.2032" layer="1" curve="90"/>
 <wire x1="16.51" y1="40.64" x2="14.859" y2="40.64" width="0.2032" layer="16"/>
 <wire x1="14.859" y1="40.64" x2="13.208" y2="42.291" width="0.2032" layer="16"/>
@@
 <contactref element="Q3" pad="1"/>
 <contactref element="R5" pad="2"/>
-<wire x1="12.33" y1="46.228" x2="12.33" y2="43.918" width="0.2032" layer="1"/>
+<wire x1="12.33" y1="46.101" x2="12.33" y2="43.918" width="0.2032" layer="1"/>
 <wire x1="12.33" y1="43.918" x2="12.53" y2="43.718" width="0.2032" layer="1" curve="90"/>
 <wire x1="16.51" y1="43.18" x2="13.068" y2="43.18" width="0.2032" layer="1"/>

Commit message: new cam, both cutouts
Parts:
- moved R6 0.13 mm to (6.35, 46.0)
Other:
- outline, holes or cut-outs redrawn
Changed lines of the file:
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@@
 <setting verticaltext="up"/>
 </settings>
-<grid distance="25" unitdist="mil" unit="mil" style="lines" multiple="1" display="yes" altdistance="1" altunitdist="mil" altunit="mil"/>
+<grid distance="50" unitdist="mil" unit="mil" style="lines" multiple="1" display="no" altdistance="5" altunitdist="mil" altunit="mil"/>
 <layers>
 <layer number="1" name="Top" color="4" fill="1" visible="yes" active="yes"/>
@@
 <layer number="14" name="Route14" color="1" fill="6" visible="no" active="no"/>
 <layer number="15" name="Route15" color="4" fill="6" visible="no" active="no"/>
-<layer number="16" name="Bottom" color="1" fill="1" visible="no" active="yes"/>
+<layer number="16" name="Bottom" color="1" fill="1" visible="yes" active="yes"/>
 <layer number="17" name="Pads" color="2" fill="1" visible="yes" active="yes"/>
 <layer number="18" name="Vias" color="2" fill="1" visible="yes" active="yes"/>
-<layer number="19" name="Unrouted" color="6" fill="1" visible="no" active="yes"/>
+<layer number="19" name="Unrouted" color="6" fill="1" visible="yes" active="yes"/>
 <layer number="20" name="Dimension" color="15" fill="1" visible="yes" active="yes"/>
 <layer number="21" name="tPlace" color="7" fill="1" visible="yes" active="yes"/>
@@
 <layer number="36" name="bGlue" color="7" fill="5" visible="no" active="yes"/>
 <layer number="37" name="tTest" color="7" fill="1" visible="no" active="yes"/>
-<layer number="38" name="bTest" color="7" fill="1" visible="no" active="yes"/>
+<layer number="38" name="bTest" color="7" fill="1" visible="yes" active="yes"/>
 <layer number="39" name="tKeepout" color="4" fill="11" visible="no" active="yes"/>
 <layer number="40" name="bKeepout" color="1" fill="11" visible="no" active="yes"/>
@@
 <layer number="44" name="Drills" color="7" fill="1" visible="no" active="yes"/>
 <layer number="45" name="Holes" color="7" fill="1" visible="no" active="yes"/>
-<layer number="46" name="Milling" color="3" fill="1" visible="no" active="yes"/>
+<layer number="46" name="Milling" color="3" fill="1" visible="yes" active="yes"/>
 <layer number="47" name="Measures" color="7" fill="1" visible="no" active="yes"/>
 <layer number="48" name="Document" color="7" fill="1" visible="no" active="yes"/>
@@
 <dimension x1="20.32" y1="49.53" x2="20.32" y2="0" x3="26.035" y3="24.765" textsize="1.778" layer="51"/>
 <text x="13.2842" y="48.133" size="1.016" layer="21" rot="R180">v1.5</text>
+<wire x1="-1.27" y1="49.53" x2="19.05" y2="49.53" width="0.1524" layer="46"/>
+<wire x1="19.05" y1="49.53" x2="19.05" y2="0" width="0.1524" layer="46"/>
+<wire x1="19.05" y1="0" x2="-1.27" y2="0" width="0.1524" layer="46"/>
+<wire x1="-1.27" y1="0" x2="-1.27" y2="49.53" width="0.1524" layer="46"/>
 </plain>
 <attributes>
@@
 <attribute name="VALUE" x="10.414" y="44.704" size="0.4064" layer="27"/>
 </element>
-<element name="R6" library="ATTAMI-V0.00" package="0805" value="" x="6.35" y="46.101" smashed="yes">
-<attribute name="VALUE" x="5.334" y="44.704" size="0.4064" layer="27"/>
+<element name="R6" library="ATTAMI-V0.00" package="0805" value="" x="6.35" y="45.974" smashed="yes">
+<attribute name="VALUE" x="5.334" y="44.577" size="0.4064" layer="27"/>
 </element>
 <element name="MOSFET-34" library="nano24rf" package="FATFAD4-LONG" value="FATPAD4LONG" x="18.1102" y="5.1816" smashed="yes" rot="R90"/>
@@
 <contactref element="RF24" pad="6"/>
 <polygon width="0.2032" layer="1">
-<vertex x="-2.54" y="49.53"/>
-<vertex x="-2.54" y="0"/>
-<vertex x="20.955" y="0"/>
-<vertex x="20.32" y="49.53"/>
+<vertex x="1.27" y="49.53"/>
+<vertex x="1.27" y="0"/>
+<vertex x="16.51" y="0"/>
+<vertex x="16.51" y="49.53"/>
 </polygon>
 <wire x1="16.51" y1="20.32" x2="9.525" y2="20.32" width="0.2032" layer="1"/>
@@
 <wire x1="-1.27" y1="15.24" x2="1.27" y2="15.24" width="1.016" layer="16"/>
 <contactref element="MOSFET-34" pad="P$4"/>
+<wire x1="16.51" y1="20.32" x2="19.05" y2="20.32" width="0" layer="19" extent="1-1"/>
 </signal>
 <signal name="FET01">
@@
 <wire x1="9.017" y1="33.528" x2="8.89" y2="33.401" width="0.2032" layer="1"/>
 <polygon width="0.2032" layer="16">
-<vertex x="-2.54" y="49.657"/>
-<vertex x="-2.54" y="0"/>
-<vertex x="21.082" y="0"/>
-<vertex x="20.4978" y="49.7332"/>
+<vertex x="1.27" y="49.657"/>
+<vertex x="1.27" y="0"/>
+<vertex x="16.51" y="0"/>
+<vertex x="16.51" y="49.53"/>
 </polygon>
 <wire x1="8.89" y1="33.401" x2="8.89" y2="33.02" width="0.3048" layer="1"/>
@@
 <contactref element="R6" pad="2"/>
 <wire x1="7.45" y1="43.718" x2="7.45" y2="46.028" width="0.2032" layer="1"/>
-<wire x1="7.45" y1="46.028" x2="7.25" y2="46.101" width="0.2032" layer="1" curve="90"/>
+<wire x1="7.45" y1="46.028" x2="7.25" y2="45.974" width="0.2032" layer="1" curve="90"/>
 <wire x1="16.51" y1="40.64" x2="14.859" y2="40.64" width="0.2032" layer="16"/>
 <wire x1="14.859" y1="40.64" x2="13.208" y2="42.291" width="0.2032" layer="16"/>
